File: pcb/touch-n-drink.kicad_sch (KiCad schematic)
At the start: 13 parts, among them J1 Display, J2 NFC, J3 Keypad, Q1 S8550, U1 ESP32-C3 SuperMini

Commit message: Update PCB project to KiCad 9.0
Changed lines of the file:
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@@
 (kicad_sch
-	(version 20231120)
+	(version 20250114)
 	(generator "eeschema")
-	(generator_version "8.0")
+	(generator_version "9.0")
 	(paper "A4")
 	(title_block
@@
 	(label "KP_Col2"
 		(at 191.77 33.02 0)
-		(fields_autoplaced yes)
 		(effects
 			(font
@@
 	(label "KP_Row4"
 		(at 118.11 59.69 0)
-		(fields_autoplaced yes)
 		(effects
 			(font
@@
 	(label "KP_Col1"
 		(at 64.77 52.07 0)
-		(fields_autoplaced yes)
 		(effects
 			(font
@@
 	(label "NFC_IRQ"
 		(at 64.77 67.31 0)
-		(fields_autoplaced yes)
 		(effects
 			(font
@@
 	(label "SDA"
 		(at 64.77 62.23 0)
-		(fields_autoplaced yes)
 		(effects
 			(font
@@
 	(label "KP_Row3"
 		(at 118.11 62.23 0)
-		(fields_autoplaced yes)
 		(effects
 			(font
@@
 	(label "KP_Col3"
 		(at 191.77 30.48 0)
-		(fields_autoplaced yes)
 		(effects
 			(font
@@
 	(label "NFC_IRQ"
 		(at 165.1 35.56 0)
-		(fields_autoplaced yes)
 		(effects
 			(font
@@
 	(label "KP_Row2"
 		(at 118.11 64.77 0)
-		(fields_autoplaced yes)
 		(effects
 			(font
@@
 	(label "KP_Col1"
 		(at 191.77 35.56 0)
-		(fields_autoplaced yes)
 		(effects
 			(font
@@
 	(label "SCL"
 		(at 165.1 40.64 0)
-		(fields_autoplaced yes)
 		(effects
 			(font
@@
 	(label "KP_Row1"
 		(at 191.77 45.72 0)
-		(fields_autoplaced yes)
 		(effects
 			(font
@@
 	(label "SCL"
 		(at 64.77 64.77 0)
-		(fields_autoplaced yes)
 		(effects
 			(font
@@
 	(label "KP_Row4"
 		(at 191.77 38.1 0)
-		(fields_autoplaced yes)
 		(effects
 			(font
@@
 	(label "SCL"
 		(at 139.7 40.64 0)
-		(fields_autoplaced yes)
 		(effects
 			(font
@@
 	(label "KP_Col3"
 		(at 64.77 57.15 0)
-		(fields_autoplaced yes)
 		(effects
 			(font
@@
 	(label "KP_Row3"
 		(at 191.77 40.64 0)
-		(fields_autoplaced yes)
 		(effects
 			(font
@@
 	(label "BUZZ"
 		(at 149.86 74.93 0)
-		(fields_autoplaced yes)
 		(effects
 			(font
@@
 	(label "KP_Row1"
 		(at 118.11 67.31 0)
-		(fields_autoplaced yes)
 		(effects
 			(font
@@
 	(label "KP_Row2"
 		(at 191.77 43.18 0)
-		(fields_autoplaced yes)
 		(effects
 			(font
@@
 	(label "KP_Col2"
 		(at 64.77 54.61 0)
-		(fields_autoplaced yes)
 		(effects
 			(font
@@
 	(label "BUZZ"
 		(at 121.92 57.15 0)
-		(fields_autoplaced yes)
 		(effects
 			(font
@@
 	(label "SDA"
 		(at 139.7 38.1 0)
-		(fields_autoplaced yes)
 		(effects
 			(font
@@
 	(label "SDA"
 		(at 165.1 38.1 0)
-		(fields_autoplaced yes)
 		(effects
 			(font
@@
 		)
 	)
+	(embedded_fonts no)
 )
